Commit message: fix: update lidar link values in go2_description.urdf and adjust parameters for laserscan

File: packages/go2_description/urdf/go2_description.urdf (robot description, URDF)
Before this commit: robot go2_description, 29 links, 28 joints
Joints:
- joint radar_joint: origin xyz=0.28945 0 -0.046825 rpy=0 2.8782 0 -> xyz=0.28945 0 -0.046825 rpy=-2.913 -0.132 -1.057
