Commit message: Refactor Unitree GO2 robot description and leg model
- Removed duplicate urdf folder
- Update with changes from Sogeti
  - Use mesh folder from Sogeti.
  - Use xacro from from Sogeti. (extra changes made to gazebo.xacro for use with gazebo harmonic and removed extra sensors not on the go2 by default)
- Removed duplicate mesh folder dae
- Removed duplicate description folder urdf

File: robotics_modules/mobile_bases/unitree_go2/go2_description/xacro/gazebo.xacro (robot description, xacro)
@@ -1,139 +1,235 @@
 <?xml version="1.0"?>
-<robot>
-    <!-- ros_control plugin -->
-    <gazebo>
-        <plugin name="gazebo_ros_control" filename="libgazebo_ros_control.so">
-            <robotNamespace>/go2_gazebo</robotNamespace>
-            <robotSimType>gazebo_ros_control/DefaultRobotHWSim</robotSimType>
+<robot xmlns:xacro="http://www.ros.org/wiki/xacro">
+    <xacro:arg name="namespace" default="" />
+    <xacro:arg name="ros_control_config_file" default="$(find go2_description)/config/ros_control.yaml" />
+    <!-- =========================================== -->
+    <!-- SENSORS SYSTEM (Required for all sensors)   -->
+    <!-- Must be loaded first for LiDAR/IMU to work  -->
+    <!-- If the gazebo world already loads a render  -->
+    <!-- engine comment out                          -->
+    <!-- =========================================== -->
+    <gazebo>
+        <plugin filename="gz-sim-sensors-system" name="gz::sim::systems::Sensors">
+            <render_engine>ogre2</render_engine>
         </plugin>
     </gazebo>
-    <!-- Show the trajectory of trunk center. -->
-    <!--gazebo>
-        <plugin name="3dplot" filename="libLinkPlot3DPlugin.so">
-            <frequency>10</frequency>
-            <plot>
-                <link>base</link>
-                <pose>0 0 0 0 0 0</pose>
-                <material>Gazebo/Yellow</material>
-            </plot>
+    <!-- =========================================== -->
+    <!-- JOINT STATE PUBLISHER (Gazebo Harmonic)     -->
+    <!-- =========================================== -->
+    <gazebo>
+        <plugin filename="gz-sim-joint-state-publisher-system"
+                name="gz::sim::systems::JointStatePublisher">
+            <!-- Front Left leg -->
+            <joint_name>FL_hip_joint</joint_name>
+            <joint_name>FL_thigh_joint</joint_name>
+            <joint_name>FL_calf_joint</joint_name>
+            <!-- Front Right leg -->
+            <joint_name>FR_hip_joint</joint_name>
+            <joint_name>FR_thigh_joint</joint_name>
+            <joint_name>FR_calf_joint</joint_name>
+            <!-- Rear Left leg -->
+            <joint_name>RL_hip_joint</joint_name>
+            <joint_name>RL_thigh_joint</joint_name>
+            <joint_name>RL_calf_joint</joint_name>
+            <!-- Rear Right leg -->
+            <joint_name>RR_hip_joint</joint_name>
+            <joint_name>RR_thigh_joint</joint_name>
+            <joint_name>RR_calf_joint</joint_name>
+            <topic>joint_states</topic>
+            <update_rate>100</update_rate>
         </plugin>
-    </gazebo-->
-    <!-- Show the trajectory of foot. You can add another trajectory about another foot. -->
-     <gazebo>
-        <plugin name="3dplot" filename="libLinkPlot3DPlugin.so">
-            <frequency>100</frequency>
-            <plot>
-                <link>FL_foot</link>
-                <pose>0 0 0 0 0 0</pose>
-            </plot>
+    </gazebo>
+    <!-- =========================================== -->
+    <!-- JOINT POSITION CONTROLLER (Gazebo Harmonic) -->
+    <!-- With PID gains to hold standing pose        -->
+    <!-- =========================================== -->
+    <gazebo>
+      <plugin filename="gz_ros2_control-system" name="gz_ros2_control::GazeboSimROS2ControlPlugin">
+      <ros>
+        <namespace>$(arg namespace)</namespace>
+      </ros>
+        <parameters>$(arg ros_control_config_file)</parameters>
+      </plugin>
+    </gazebo>
+    <!-- =========================================== -->
+    <!-- ODOMETRY PUBLISHER (Gazebo Harmonic)        -->
+    <!-- For legged robot odometry estimation        -->
+    <!-- =========================================== -->
+    <gazebo>
+        <plugin filename="gz-sim-odometry-publisher-system"
+                name="gz::sim::systems::OdometryPublisher">
+            <odom_frame>odom</odom_frame>
+            <robot_base_frame>base_link</robot_base_frame>
+            <odom_publish_frequency>50</odom_publish_frequency>
+            <odom_topic>$(arg namespace)/odom</odom_topic>
+            <!-- 3D odometry for legged robot -->
+            <dimensions>3</dimensions>
         </plugin>
     </gazebo>
-    <gazebo>
-        <plugin filename="libgazebo_ros_force.so" name="gazebo_ros_force">
-            <bodyName>trunk</bodyName>
-            <topicName>/apply_force/trunk</topicName>
-        </plugin>
+    <!-- =========================================== -->
+    <!-- IMU SENSOR - Gazebo Harmonic Format         -->
+    <!-- =========================================== -->
+    <gazebo>
+    <plugin filename="gz-sim-imu-system" name="gz::sim::systems::Imu"> </plugin>
     </gazebo>
     <gazebo reference="imu_link">
-        <gravity>true</gravity>
         <sensor name="imu_sensor" type="imu">
             <always_on>true</always_on>
-            <update_rate>1000</update_rate>
+            <update_rate>60</update_rate>
             <visualize>true</visualize>
-            <topic>__default_topic__</topic>
-            <plugin filename="libgazebo_ros_imu_sensor.so" name="imu_plugin">
-                <topicName>trunk_imu</topicName>
-                <bodyName>imu_link</bodyName>
-                <updateRateHZ>1000.0</updateRateHZ>
-                <gaussianNoise>0.0</gaussianNoise>
-                <xyzOffset>0 0 0</xyzOffset>
-                <rpyOffset>0 0 0</rpyOffset>
-                <frameName>imu_link</frameName>
-            </plugin>
-            <pose>0 0 0 0 0 0</pose>
-        </sensor>
-    </gazebo>
-    <!-- Foot contacts. -->
-    <gazebo reference="FR_calf">
+            <topic>$(arg namespace)/imu</topic>
+            <gz_frame_id>imu_link</gz_frame_id>
+            <imu>
+                <enable_orientation>1</enable_orientation>
+                <angular_velocity>
+                    <x>
+                        <noise type="gaussian">
+                            <mean>0.0</mean>
+                            <stddev>2e-4</stddev>
+                        </noise>
+                    </x>
+                    <y>
+                        <noise type="gaussian">
+                            <mean>0.0</mean>
+                            <stddev>2e-4</stddev>
+                        </noise>
+                    </y>
+                    <z>
+                        <noise type="gaussian">
+                            <mean>0.0</mean>
+                            <stddev>2e-4</stddev>
+                        </noise>
+                    </z>
+                </angular_velocity>
+                <linear_acceleration>
+                    <x>
+                        <noise type="gaussian">
+                            <mean>0.0</mean>
+                            <stddev>1.7e-2</stddev>
+                        </noise>
+                    </x>
+                    <y>
+                        <noise type="gaussian">
+                            <mean>0.0</mean>
+                            <stddev>1.7e-2</stddev>
+                        </noise>
+                    </y>
+                    <z>
+                        <noise type="gaussian">
+                            <mean>0.0</mean>
+                            <stddev>1.7e-2</stddev>
+                        </noise>
+                    </z>
+                </linear_acceleration>
+            </imu>
+        </sensor>
+    </gazebo>
+    <!-- =========================================== -->
+    <!-- FRONT CAMERA SENSOR (Gazebo Harmonic)       -->
+    <!-- =========================================== -->
+    <gazebo reference="front_camera_link">
+        <sensor name="front_camera" type="camera">
+            <always_on>true</always_on>
+            <update_rate>30</update_rate>
+            <visualize>false</visualize>
+            <topic>front_camera/image_raw</topic>
+            <camera name="front_camera">
+                <horizontal_fov>1.5708</horizontal_fov>
+                <image>
+                    <width>640</width>
+                    <height>480</height>
+                    <format>R8G8B8</format>
+                </image>
+                <clip>
+                    <near>0.05</near>
+                    <far>100</far>
+                </clip>
+                <noise>
+                    <type>gaussian</type>
+                    <mean>0.0</mean>
+                    <stddev>0.007</stddev>
+                </noise>
+            </camera>
+        </sensor>
+    </gazebo>
+    <!-- =========================================== -->
+    <!-- FOOT CONTACT SENSORS (Gazebo Harmonic)      -->
+    <!-- =========================================== -->
+    <gazebo reference="FL_foot">
+        <sensor name="FL_foot_contact" type="contact">
+            <always_on>true</always_on>
+            <update_rate>100</update_rate>
+            <contact>
+                <collision>FL_foot_collision</collision>
+            </contact>
+            <topic>FL_foot_contact</topic>
+        </sensor>
+    </gazebo>
+    <gazebo reference="FR_foot">
         <sensor name="FR_foot_contact" type="contact">
-        <update_rate>100</update_rate>
-        <plugin name="contactPlugin" filename="libunitreeFootContactPlugin.so"/>
-        <contact>
-            <collision>FR_calf_fixed_joint_lump__FR_foot_collision_1</collision>
-        </contact>
-        </sensor>
-    </gazebo>
-    <gazebo reference="FL_calf">
-        <sensor name="FL_foot_contact" type="contact">
-        <update_rate>100</update_rate>
-        <plugin name="contactPlugin" filename="libunitreeFootContactPlugin.so"/>
-        <contact>
-            <collision>FL_calf_fixed_joint_lump__FL_foot_collision_1</collision>
-        </contact>
-        </sensor>
-    </gazebo>
-    <gazebo reference="RR_calf">
+            <always_on>true</always_on>
+            <update_rate>100</update_rate>
+            <contact>
+                <collision>FR_foot_collision</collision>
+            </contact>
+            <topic>FR_foot_contact</topic>
+        </sensor>
+    </gazebo>
+    <gazebo reference="RL_foot">
+        <sensor name="RL_foot_contact" type="contact">
+            <always_on>true</always_on>
+            <update_rate>100</update_rate>
+            <contact>
+                <collision>RL_foot_collision</collision>
+            </contact>
+            <topic>RL_foot_contact</topic>
+        </sensor>
+    </gazebo>
+    <gazebo reference="RR_foot">
         <sensor name="RR_foot_contact" type="contact">
-        <update_rate>100</update_rate>
-        <plugin name="contactPlugin" filename="libunitreeFootContactPlugin.so"/>
-        <contact>
-            <collision>RR_calf_fixed_joint_lump__RR_foot_collision_1</collision>
-        </contact>
-        </sensor>
-    </gazebo>
-    <gazebo reference="RL_calf">
-        <sensor name="RL_foot_contact" type="contact">
-        <update_rate>100</update_rate>
-        <plugin name="contactPlugin" filename="libunitreeFootContactPlugin.so"/>
-        <contact>
-            <collision>RL_calf_fixed_joint_lump__RL_foot_collision_1</collision>
-        </contact>
-        </sensor>
-    </gazebo>
-    <!-- Visualization of Foot contacts. -->
-    <gazebo reference="FR_foot">
-        <visual>
-            <plugin name="drawForcePlugin" filename="libunitreeDrawForcePlugin.so">
-                <topicName>FR_foot_contact</topicName>
-            </plugin>
-        </visual>
-    </gazebo>
-    <gazebo reference="FL_foot">
-        <visual>
-            <plugin name="drawForcePlugin" filename="libunitreeDrawForcePlugin.so">
-                <topicName>FL_foot_contact</topicName>
-            </plugin>
-        </visual>
-    </gazebo>
-    <gazebo reference="RR_foot">
-        <visual>
-            <plugin name="drawForcePlugin" filename="libunitreeDrawForcePlugin.so">
-                <topicName>RR_foot_contact</topicName>
-            </plugin>
-        </visual>
-    </gazebo>
-    <gazebo reference="RL_foot">
-        <visual>
-            <plugin name="drawForcePlugin" filename="libunitreeDrawForcePlugin.so">
-                <topicName>RL_foot_contact</topicName>
-            </plugin>
-        </visual>
-    </gazebo>
-    <gazebo reference="base">
-        <turnGravityOff>false</turnGravityOff>
+            <always_on>true</always_on>
+            <update_rate>100</update_rate>
+            <contact>
+                <collision>RR_foot_collision</collision>
+            </contact>
+            <topic>RR_foot_contact</topic>
+        </sensor>
+    </gazebo>
+    <!-- =========================================== -->
+    <!-- GAZEBO MATERIALS AND PHYSICS                -->
+    <!-- =========================================== -->
+    <gazebo reference="base_link">
+        <self_collide>false</self_collide>
     </gazebo>
     <gazebo reference="trunk">
         <mu1>0.2</mu1>
         <mu2>0.2</mu2>
-        <kp  value="1000000.0"/>
-        <kd  value="1.0"/>
-    </gazebo>
-    <gazebo reference="stick_link">
-        <mu1>0.2</mu1>
-        <mu2>0.2</mu2>
+        <kp>1000000.0</kp>
+        <kd>1.0</kd>
+        <self_collide>false</self_collide>
+        <material>
+            <ambient>0.5 0.5 0.5 1</ambient>
+            <diffuse>0.5 0.5 0.5 1</diffuse>
+        </material>
     </gazebo>
     <gazebo reference="imu_link">
         <mu1>0.2</mu1>
         <mu2>0.2</mu2>
+        <material>
+            <ambient>1.0 0.5 0.0 1</ambient>
+            <diffuse>1.0 0.5 0.0 1</diffuse>
+        </material>
+    </gazebo>
+    <gazebo reference="front_camera_link">
+        <material>
+            <ambient>0.3 0.3 0.3 1</ambient>
+            <diffuse>0.3 0.3 0.3 1</diffuse>
+        </material>
+    </gazebo>
+    <gazebo reference="radar_link">
+        <material>
+            <ambient>0.1 0.1 0.1 1</ambient>
+            <diffuse>0.1 0.1 0.1 1</diffuse>
+        </material>
     </gazebo>
     <!-- FL leg -->
@@ -141,23 +237,24 @@
         <mu1>0.2</mu1>
         <mu2>0.2</mu2>
+        <self_collide>false</self_collide>
     </gazebo>
     <gazebo reference="FL_thigh">
         <mu1>0.2</mu1>
         <mu2>0.2</mu2>
-        <self_collide>1</self_collide>
-        <kp  value="1000000.0"/>
-        <kd  value="1.0"/>
+        <self_collide>true</self_collide>
+        <kp>1000000.0</kp>
+        <kd>1.0</kd>
     </gazebo>
     <gazebo reference="FL_calf">
         <mu1>0.2</mu1>
         <mu2>0.2</mu2>
-        <self_collide>1</self_collide>
+        <self_collide>true</self_collide>
     </gazebo>
     <gazebo reference="FL_foot">
-        <mu1>0.6</mu1>
-        <mu2>0.6</mu2>
-        <self_collide>1</self_collide>
-        <kp  value="1000000.0"/>
-        <kd  value="1.0"/>
+        <mu1>0.8</mu1>
+        <mu2>0.8</mu2>
+        <self_collide>true</self_collide>
+        <kp>1000000.0</kp>
+        <kd>1.0</kd>
     </gazebo>
     <!-- FR leg -->
@@ -165,23 +262,24 @@
         <mu1>0.2</mu1>
         <mu2>0.2</mu2>
+        <self_collide>false</self_collide>
     </gazebo>
     <gazebo reference="FR_thigh">
         <mu1>0.2</mu1>
         <mu2>0.2</mu2>
-        <self_collide>1</self_collide>
-        <kp  value="1000000.0"/>
-        <kd  value="1.0"/>
+        <self_collide>true</self_collide>
+        <kp>1000000.0</kp>
+        <kd>1.0</kd>
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
File: robotics_modules/mobile_bases/unitree_go2/go2_description/xacro/leg.xacro (robot description, xacro)
@@ -27,4 +27,20 @@
             </xacro:if>
         </joint>
+        <joint name="${name}_hip_rotor_joint" type="fixed">
+            <xacro:if value="${(mirror_dae == False) and (front_hind_dae == True)}">
+                <origin rpy="0 0 0" xyz="${hip_rotor_offset_x} ${-hip_rotor_offset_y} 0"/>
+            </xacro:if>
+            <xacro:if value="${(mirror_dae == True) and (front_hind_dae == True)}">
+                <origin rpy="0 0 0" xyz="${hip_rotor_offset_x} ${hip_rotor_offset_y} 0"/>
+            </xacro:if>
+            <xacro:if value="${(mirror_dae == False) and (front_hind_dae == False)}">
+                <origin rpy="0 0 0" xyz="${-hip_rotor_offset_x} ${-hip_rotor_offset_y} 0"/>
+            </xacro:if>
+            <xacro:if value="${(mirror_dae == True) and (front_hind_dae == False)}">
+                <origin rpy="0 0 0" xyz="${-hip_rotor_offset_x} ${hip_rotor_offset_y} 0"/>
+            </xacro:if>
+            <parent link="trunk"/>
+            <child link="${name}_hip_rotor"/>
+        </joint>
         <link name="${name}_hip">
             <visual>
@@ -59,4 +75,27 @@
                     iyy="${hip_iyy}" iyz="${hip_iyz*mirror}"
                     izz="${hip_izz}"/>
+            </inertial>
+        </link>
+        <link name="${name}_hip_rotor">
+            <visual>
+                <origin rpy="0 ${PI/2.0} 0" xyz="0 0 0"/>
+                <geometry>
+                    <cylinder length="0.02" radius="0.035"/>
+                </geometry>
+                <material name="green"/>
+            </visual>
+            <!-- <collision>
+                <origin rpy="0 ${PI/2.0} 0" xyz="0 0 0"/>
+                <geometry>
+                    <cylinder length="0.02" radius="0.035"/>
+                </geometry>
+            </collision> -->
+            <inertial>
+                <origin rpy="0 0 0" xyz="${hip_rotor_com_x} ${hip_rotor_com_y} ${hip_rotor_com_z}"/>
+                <mass value="${hip_rotor_mass}"/>
+                <inertia
+                    ixx="${hip_rotor_ixx}" ixy="${hip_rotor_ixy}" ixz="${hip_rotor_ixz}"
+                    iyy="${hip_rotor_iyy}" iyz="${hip_rotor_iyz}"
+                    izz="${hip_rotor_izz}"/>
             </inertial>
         </link>
@@ -69,4 +108,9 @@
             <limit effort="${thigh_torque_max}" velocity="${thigh_velocity_max}" lower="${thigh_position_min}" upper="${thigh_position_max}"/>
         </joint>
+        <joint name="${name}_thigh_rotor_joint" type="fixed">
+            <origin rpy="0 0 0" xyz="${thigh_rotor_offset_x} ${thigh_rotor_offset_y*mirror} 0"/>
+            <parent link="${name}_hip"/>
+            <child link="${name}_thigh_rotor"/>
+        </joint>
         <link name="${name}_thigh">
             <visual>
@@ -95,4 +139,27 @@
                     iyy="${thigh_iyy}" iyz="${thigh_iyz*mirror}"
                     izz="${thigh_izz}"/>
+            </inertial>
+        </link>
+        <link name="${name}_thigh_rotor">
+            <visual>
+                <origin rpy="${PI/2.0} 0 0" xyz="0 0 0"/>
+                <geometry>
+                    <cylinder length="0.02" radius="0.035"/>
+                </geometry>
+                <material name="green"/>
+            </visual>
+            <!-- <collision>
+                <origin rpy="${PI/2.0} 0 0" xyz="0 0 0"/>
+                <geometry>
+                    <cylinder length="0.02" radius="0.035"/>
+                </geometry>
+            </collision> -->
+            <inertial>
+                <origin rpy="0 0 0" xyz="${thigh_rotor_com_x} ${thigh_rotor_com_y} ${thigh_rotor_com_z}"/>
+                <mass value="${thigh_rotor_mass}"/>
+                <inertia
+                    ixx="${thigh_rotor_ixx}" ixy="${thigh_rotor_ixy}" ixz="${thigh_rotor_ixz}"
+                    iyy="${thigh_rotor_iyy}" iyz="${thigh_rotor_iyz}"
+                    izz="${thigh_rotor_izz}"/>
             </inertial>
         </link>
@@ -105,9 +172,19 @@
             <limit effort="${calf_torque_max}" velocity="${calf_velocity_max}" lower="${calf_position_min}" upper="${calf_position_max}"/>
         </joint>
+        <joint name="${name}_calf_rotor_joint" type="fixed">
+            <origin rpy="0 0 0" xyz="${calf_rotor_offset_x} ${calf_rotor_offset_y*mirror} 0"/>
+            <parent link="${name}_thigh"/>
+            <child link="${name}_calf_rotor"/>
+        </joint>
         <link name="${name}_calf">
             <visual>
                 <origin rpy="0 0 0" xyz="0 0 0"/>
                 <geometry>
-                    <mesh filename="package://go2_description/meshes/calf.dae" scale="1 1 1"/>
+                    <xacro:if value="${mirror_dae == True}">
+                        <mesh filename="package://go2_description/meshes/calf.dae" scale="1 1 1"/>
+                    </xacro:if>
+                    <xacro:if value="${mirror_dae == False}">
+                        <mesh filename="package://go2_description/meshes/calf_mirror.dae" scale="1 1 1"/>
+                    </xacro:if>
                 </geometry>
                 <!-- <material name="orange"/> -->
@@ -128,5 +205,28 @@
             </inertial>
         </link>
-        <joint name="${name}_foot_fixed" type="fixed">0
+        <link name="${name}_calf_rotor">
+            <visual>
+                <origin rpy="${PI/2.0} 0 0" xyz="0 0 0"/>
+                <geometry>
+                    <cylinder length="0.02" radius="0.035"/>
+                </geometry>
+                <material name="green"/>
+            </visual>
+            <!-- <collision>
+                <origin rpy="${PI/2.0} 0 0" xyz="0 0 0"/>
+                <geometry>
+                    <cylinder length="0.02" radius="0.035"/>
+                </geometry>
+            </collision> -->
+            <inertial>
+                <origin rpy="0 0 0" xyz="${calf_rotor_com_x} ${calf_rotor_com_y} ${calf_rotor_com_z}"/>
+                <mass value="${calf_rotor_mass}"/>
+                <inertia
+                    ixx="${calf_rotor_ixx}" ixy="${calf_rotor_ixy}" ixz="${calf_rotor_ixz}"
+                    iyy="${calf_rotor_iyy}" iyz="${calf_rotor_iyz}"
+                    izz="${calf_rotor_izz}"/>
+            </inertial>
+        </link>
+        <joint name="${name}_foot_fixed" type="fixed">
             <origin rpy="0 0 0" xyz="0 0 ${-(calf_length)}"/>
             <parent link="${name}_calf"/>
