Commit message: fix: compensate Go2 body tilt and lidar mount pitch in the 2D scan
Ground showed up in /scan and the SLAM map. Measured on the robot:
- the lidar mount is ~18.5 deg pitched (Livox IMU vs Go2 IMU, and the
  ground plane in the cloud), not the 17 deg in the URDF;
- the body pitches/rolls up to +-5 deg while walking (0.8-1.7 deg when
  standing), but TF had base_footprint fixed to the body with a 2D EKF.
At 2-5 m this put the ground 10-25 cm too high, above min_height.

- New imu_tilt_tf node publishes base_footprint -> base_link with the
  roll/pitch from /imu (hardware only); the URDF drops its fixed
  base_footprint joint via xacro arg imu_tilt (simulation unchanged).
- Lidar mount pitch 17 -> 18.5 deg.
- min_height -0.25 -> -0.22 (8 cm above the ground).

Co-authored-by: Copilot <223556219+Copilot@users.noreply.github.com>

File: robotics_modules/mobile_bases/unitree_go2/go2_description/xacro/unitree_go2.xacro (robot description, xacro)
@@ -2,4 +2,7 @@
 <robot name="go2" xmlns:xacro="http://www.ros.org/wiki/xacro">
     <xacro:arg name="DEBUG" default="false"/>
+    <!-- On hardware, imu_tilt_tf.py publishes base_footprint -> base_link with
+         the body roll and pitch from the IMU, so the URDF must not. -->
+    <xacro:arg name="imu_tilt" default="false"/>
     <xacro:include filename="$(find go2_description)/xacro/constants.xacro"/>
     <xacro:include filename="$(find go2_description)/xacro/materials.xacro"/>
@@ -22,12 +25,14 @@
         <!-- No inertia, no mass - this is just a reference frame -->
     </link>
-     <link name="base_footprint">
-        <!-- No inertia, no mass - this is just a reference frame -->
-    </link>
-    <joint name="base_to_footprint" type="fixed">
-        <origin rpy="0 0 0" xyz="0 0 0"/>
-        <parent link="base_footprint"/>
-        <child link="base_link"/>
-    </joint>
+    <xacro:unless value="$(arg imu_tilt)">
+        <link name="base_footprint">
+            <!-- No inertia, no mass - this is just a reference frame -->
+        </link>
+        <joint name="base_to_footprint" type="fixed">
+            <origin rpy="0 0 0" xyz="0 0 0"/>
+            <parent link="base_footprint"/>
+            <child link="base_link"/>
+        </joint>
+    </xacro:unless>
     <!--
         Fixed joint connecting base_link to the actual robot body (trunk).

File: robotics_modules/platform_kits/enexis_go2/xacro/enexis_go2.xacro (robot description, xacro)
@@ -4,9 +4,10 @@
     <xacro:include filename="$(find septentrio)/xacro/gnss.xacro"/>
     <xacro:include filename="$(find go2_description)/xacro/unitree_go2.xacro"/>
-    <!-- Joint attaching lidar to trunk (mounted on top) -->
+    <!-- Joint attaching lidar to trunk (mounted on top). The 18.5 deg pitch was
+         measured on the robot (Livox IMU vs Go2 IMU); the drawing value is 17 deg. -->
     <joint name="lidar_joint" type="fixed">
         <parent link="trunk"/>
         <child link="lidar_link"/>
-        <origin xyz="0.32 0.0 ${trunk_height/2.0 + lidar_height/2.0 + 0.051}" rpy="0 ${17*pi/180} 0"/>
+        <origin xyz="0.32 0.0 ${trunk_height/2.0 + lidar_height/2.0 + 0.051}" rpy="0 ${18.5*pi/180} 0"/>
     </joint>
     <joint name="gps_joint" type="fixed">
