Commit message: feat: add septentrio to enexis_go2 platform kit

File: robotics_modules/platform_kits/enexis_go2/xacro/enexis_go2.xacro (robot description, xacro)
@@ -2,5 +2,5 @@
 <robot name="go2" xmlns:xacro="http://www.ros.org/wiki/xacro">
     <xacro:include filename="$(find sim_lidar)/xacro/lidar.xacro"/>
-    <xacro:include filename="$(find sim_gnss)/xacro/gnss.xacro"/>
+    <xacro:include filename="$(find septentrio)/xacro/gnss.xacro"/>
     <xacro:include filename="$(find go2_description)/xacro/unitree_go2.xacro"/>
     <!-- Joint attaching lidar to trunk (mounted on top) -->
@@ -14,5 +14,10 @@
         <parent link="trunk"/>
         <child link="gps_link"/>
-        <origin xyz="0 0 0" rpy="0 0 0"/>
+        <origin xyz="0.325 0 0" rpy="0 0 0"/>
+    </joint>
+    <joint name="aux_gps_joint" type="fixed">
+        <parent link="trunk"/>
+        <child link="aux_gps_link"/>
+        <origin xyz="-0.11 0 0" rpy="0 0 0"/>
     </joint>
 </robot>

Commit message: fix: update lidar joint position and orientation in enexis_go2.xacro

File: robotics_modules/platform_kits/enexis_go2/xacro/enexis_go2.xacro (robot description, xacro)
@@ -8,6 +8,5 @@
         <parent link="trunk"/>
         <child link="lidar_link"/>
-        <!-- Positioned on top of the trunk, centered -->
-        <origin xyz="0.22 0.0 ${trunk_height/2.0 + lidar_height/2.0 + 0.051}" rpy="0 0 0"/>
+        <origin xyz="0.32 0.0 ${trunk_height/2.0 + lidar_height/2.0 + 0.051}" rpy="0 ${17*pi/180} 0"/>
     </joint>
     <joint name="gps_joint" type="fixed">
