Commit message: fix: take EKF yaw rate from the offset-corrected Livox gyro
Heading drifted while mapping. Measured on the robot (90 s of turning,
scan matching as reference):
- the Go2 /imu gyro has a constant 0.34 deg/s offset, which the local EKF
  integrated uncorrected: ~20 deg/min of drift while standing still;
- it also reads turns ~3% too large (361 deg for a 354 deg turn);
- the Livox gyro agrees with scan matching within ~1% and has a smaller,
  equally stable offset (0.13 deg/s).

- New gyro_bias_correction node republishes /livox/imu as
  /livox/imu_corrected: learns the gyro offset at standstill (low gyro
  noise, no non-zero /cmd_vel for 1.5 s), subtracts it, and converts the
  Livox acceleration from g to m/s^2.
- localization.launch.py livox_gyro:=True (hardware compose) feeds it to
  the local EKF as imu0, with a 50 ms transform_timeout for the IMU-driven
  tilt TF. Simulation keeps /imu.
- livox_frame (Livox IMU frame) attached to lidar_link in the URDF.

Co-authored-by: Copilot <223556219+Copilot@users.noreply.github.com>

File: robotics_modules/platform_kits/enexis_go2/xacro/enexis_go2.xacro (robot description, xacro)
@@ -11,4 +11,12 @@
         <origin xyz="0.32 0.0 ${trunk_height/2.0 + lidar_height/2.0 + 0.051}" rpy="0 ${18.5*pi/180} 0"/>
     </joint>
+    <!-- The Livox driver publishes /livox/imu in livox_frame. MID360 IMU offset
+         from the point cloud origin, axes aligned (Livox MID360 user manual). -->
+    <link name="livox_frame"/>
+    <joint name="livox_imu_joint" type="fixed">
+        <parent link="lidar_link"/>
+        <child link="livox_frame"/>
+        <origin xyz="0.011 0.02329 -0.04412" rpy="0 0 0"/>
+    </joint>
     <joint name="gps_joint" type="fixed">
         <parent link="trunk"/>
